Commit message: working w final legs?

File: body.urdf (robot description, URDF)
Before this commit: robot robot, 3 links, 2 joints
Links:
- added link BackLowerleg, mass 1; collision box size=0.2 0.2 1; visual box size=0.2 0.2 1
- added link FrontLowerleg, mass 1; collision box size=0.2 0.2 1; visual box size=0.2 0.2 1
- added link LeftLowerleg, mass 1; collision box size=0.2 0.2 1; visual box size=0.2 0.2 1
- added link Leftleg, mass 1; collision box size=1 0.2 0.2; visual box size=1 0.2 0.2
- added link RightLowerleg, mass 1; collision box size=0.2 0.2 1; visual box size=0.2 0.2 1
- added link Rightleg, mass 1; collision box size=1 0.2 0.2; visual box size=1 0.2 0.2
- link BackLeg: geometry collision box size=0.2 1 0.2; visual box size=0.2 1 0.2
- link FrontLeg: geometry collision box size=0.2 1 0.2; visual box size=0.2 1 0.2
Joints:
- added joint Backleg_BacklowerLeg: type revolute, parent Backleg, child BackLowerleg, origin xyz=0 -0.5 0 rpy=0 0 0, axis 1 0 0, limit lower=-3.14159 upper=3.14159 effort=0.0 velocity=0.0
- added joint Frontleg_FrontlowerLeg: type revolute, parent FrontLeg, child FrontLowerleg, origin xyz=0 1 0 rpy=0 0 0, axis 1 0 0, limit lower=-3.14159 upper=3.14159 effort=0.0 velocity=0.0
- added joint Leftleg_Leftlowerleg: type revolute, parent Leftleg, child LeftLowerleg, origin xyz=-0.5 0 0 rpy=0 0 0, axis 1 0 0, limit lower=-3.14159 upper=3.14159 effort=0.0 velocity=0.0
- added joint Rightleg_RightLowerleg: type revolute, parent Rightleg, child RightLowerleg, origin xyz=0.5 0 0 rpy=0 0 0, axis 1 0 0, limit lower=-3.14159 upper=3.14159 effort=0.0 velocity=0.0
- added joint Torso_LeftLeg: type revolute, parent Torso, child Leftleg, origin xyz=-0.5 0 1 rpy=0 0 0, axis 1 0 0, limit lower=-3.14159 upper=3.14159 effort=0.0 velocity=0.0
- added joint Torso_RightLeg: type revolute, parent Torso, child Rightleg, origin xyz=0.5 0 1 rpy=0 0 0, axis 1 0 0, limit lower=-3.14159 upper=3.14159 effort=0.0 velocity=0.0
- joint Torso_BackLeg: axis 0 1 0 -> 1 0 0; origin xyz=1 0 1 rpy=0 0 0 -> xyz=0 -0.5 1 rpy=0 0 0
- joint Torso_FrontLeg: axis 0 1 0 -> 1 0 0; origin xyz=2 0 1 rpy=0 0 0 -> xyz=0 0.5 1 rpy=0 0 0

Commit message: working, the front leg is not attatched

File: body.urdf (robot description, URDF)
Before this commit: robot robot, 9 links, 8 joints
Joints:
- joint Backleg_BacklowerLeg: origin xyz=0 -0.5 0 rpy=0 0 0 -> xyz=0 -1 0 rpy=0 0 0; parent Backleg -> BackLeg
- joint Leftleg_Leftlowerleg: axis 1 0 0 -> 0 1 0; origin xyz=-0.5 0 0 rpy=0 0 0 -> xyz=-1 0 0 rpy=0 0 0; parent Leftleg -> FrontLeg
- joint Rightleg_RightLowerleg: axis 1 0 0 -> 0 1 0; origin xyz=0.5 0 0 rpy=0 0 0 -> xyz=1 0 0 rpy=0 0 0
- joint Torso_LeftLeg: axis 1 0 0 -> 0 1 0
- joint Torso_RightLeg: axis 1 0 0 -> 0 1 0

Commit message: changes

File: body.urdf (robot description, URDF)
Before this commit: robot robot, 9 links, 8 joints
Joints:
- joint Leftleg_Leftlowerleg: origin xyz=-1 0 0 rpy=0 0 0 -> xyz=-1.5 -0.5 0 rpy=0 0 0

Commit message: torsorightlink

File: body.urdf (robot description, URDF)
Before this commit: robot robot, 9 links, 8 joints
Links:
- added link RightLowerlegTwo, mass 1; collision box size=0.2 0.2 1; visual box size=0.2 0.2 1
- added link RightlegTwo, mass 1; collision box size=1 0.2 0.2; visual box size=1 0.2 0.2
Joints:
- added joint Rightleg_RightLowerlegTwo: type revolute, parent Rightleg, child RightLowerlegTwo, origin xyz=1 0 0 rpy=0 0 0, axis 0 1 0, limit lower=-3.14159 upper=3.14159 effort=0.0 velocity=0.0
- added joint Torso_RightLegTwo: type revolute, parent Torso, child Rightleg, origin xyz=0.5 0 1 rpy=0 0 0, axis 0 1 0, limit lower=-3.14159 upper=3.14159 effort=0.0 velocity=0.0

Commit message: final project hexa finished

File: body.urdf (robot description, URDF)
Before this commit: robot robot, 11 links, 10 joints
Links:
- added link LeftLowerlegTwo, mass 1; collision box size=0.2 0.2 1; visual box size=0.2 0.2 1
- added link LeftlegTwo, mass 1; collision box size=1 0.2 0.2; visual box size=1 0.2 0.2
Joints:
- added joint Leftleg_LeftlowerlegTwo: type revolute, parent FrontLeg, child LeftLowerlegTwo, origin xyz=-1.5 -0.5 0 rpy=0 0 0, axis 0 1 0, limit lower=-3.14159 upper=3.14159 effort=0.0 velocity=0.0
- added joint Torso_LeftLegTwo: type revolute, parent Torso, child LeftlegTwo, origin xyz=-0.5 0 1 rpy=0 0 0, axis 0 1 0, limit lower=-3.14159 upper=3.14159 effort=0.0 velocity=0.0
- joint Torso_RightLegTwo: child Rightleg -> RightlegTwo

Commit message: no permission

File: body.urdf (robot description, URDF)
Before this commit: robot robot, 13 links, 12 joints
Links:
- removed link BackLowerleg
- removed link FrontLowerleg
- removed link LeftLowerleg
- removed link LeftLowerlegTwo
- removed link Leftleg
- removed link LeftlegTwo
- removed link RightLowerleg
- removed link RightLowerlegTwo
- removed link Rightleg
- removed link RightlegTwo
- added link BackLowerLeg, mass 1; collision box size=0.2 0.2 1; visual box size=0.2 0.2 1
- added link FrontLowerLeg, mass 1; collision box size=0.2 0.2 1; visual box size=0.2 0.2 1
- added link LeftLegFirst, mass 1; collision box size=1.0 0.2 0.2; visual box size=1.0 0.2 0.2
- added link LeftLegSecond, mass 1; collision box size=1.0 0.2 0.2; visual box size=1.0 0.2 0.2
- added link LeftLowerLegFirst, mass 1; collision box size=0.2 0.2 1; visual box size=0.2 0.2 1
- added link LeftLowerLegSecond, mass 1; collision box size=0.2 0.2 1; visual box size=0.2 0.2 1
- added link RightLegFirst, mass 1; collision box size=1.0 0.2 0.2; visual box size=1.0 0.2 0.2
- added link RightLegSecond, mass 1; collision box size=1.0 0.2 0.2; visual box size=1.0 0.2 0.2
- added link RightLowerLegFirst, mass 1; collision box size=0.2 0.2 1; visual box size=0.2 0.2 1
- added link RightLowerLegSecond, mass 1; collision box size=0.2 0.2 1; visual box size=0.2 0.2 1
Joints:
- removed joint Backleg_BacklowerLeg
- removed joint Frontleg_FrontlowerLeg
- removed joint Leftleg_Leftlowerleg
- removed joint Leftleg_LeftlowerlegTwo
- removed joint Rightleg_RightLowerleg
- removed joint Rightleg_RightLowerlegTwo
- removed joint Torso_LeftLeg
- removed joint Torso_LeftLegTwo
- removed joint Torso_RightLeg
- removed joint Torso_RightLegTwo
- added joint BackLeg_BackLowerLeg: type revolute, parent BackLeg, child BackLowerLeg, origin xyz=0 -1 0 rpy=0 0 0, axis 1 0 0, limit lower=-3.14159 upper=3.14159 effort=0.0 velocity=0.0
- added joint FrontLeg_FrontLowerLeg: type revolute, parent FrontLeg, child FrontLowerLeg, origin xyz=0 1 0 rpy=0 0 0, axis 1 0 0, limit lower=-3.14159 upper=3.14159 effort=0.0 velocity=0.0
- added joint LeftLegFirst_LeftLowerLegFirst: type revolute, parent LeftLegFirst, child LeftLowerLegFirst, origin xyz=-1 0 0 rpy=0 0 0, axis 0 1 0, limit lower=-3.14159 upper=3.14159 effort=0.0 velocity=0.0
- added joint LeftLegSecond_LeftLowerLegSecond: type revolute, parent LeftLegSecond, child LeftLowerLegSecond, origin xyz=-1 0 0 rpy=0 0 0, axis 0 1 0, limit lower=-3.14159 upper=3.14159 effort=0.0 velocity=0.0
- added joint RightLegFirst_RightLowerLegFirst: type revolute, parent RightLegFirst, child RightLowerLegFirst, origin xyz=1 0 0 rpy=0 0 0, axis 0 1 0, limit lower=-3.14159 upper=3.14159 effort=0.0 velocity=0.0
- added joint RightLegSecond_RightLowerLegSecond: type revolute, parent RightLegSecond, child RightLowerLegSecond, origin xyz=1 0 0 rpy=0 0 0, axis 0 1 0, limit lower=-3.14159 upper=3.14159 effort=0.0 velocity=0.0
- added joint Torso_LeftLegFirst: type revolute, parent Torso, child LeftLegFirst, origin xyz=-0.5 -0.1 2 rpy=0 0 0, axis 0 1 0, limit lower=-3.14159 upper=3.14159 effort=0.0 velocity=0.0
- added joint Torso_LeftLegSecond: type revolute, parent Torso, child LeftLegSecond, origin xyz=-0.5 0.1 2 rpy=0 0 0, axis 0 1 0, limit lower=-3.14159 upper=3.14159 effort=0.0 velocity=0.0
- added joint Torso_RightLegFirst: type revolute, parent Torso, child RightLegFirst, origin xyz=0.5 -0.1 2 rpy=0 0 0, axis 0 1 0, limit lower=-3.14159 upper=3.14159 effort=0.0 velocity=0.0
- added joint Torso_RightLegSecond: type revolute, parent Torso, child RightLegSecond, origin xyz=0.5 0.1 2 rpy=0 0 0, axis 0 1 0, limit lower=-3.14159 upper=3.14159 effort=0.0 velocity=0.0
- joint Torso_BackLeg: origin xyz=0 -0.5 1 rpy=0 0 0 -> xyz=0 -0.5 2 rpy=0 0 0
- joint Torso_FrontLeg: origin xyz=0 0.5 1 rpy=0 0 0 -> xyz=0 0.5 2 rpy=0 0 0

Commit message: finished

File: body.urdf (robot description, URDF)
Before this commit: robot robot, 13 links, 12 joints
Joints:
- joint Torso_BackLeg: origin xyz=0 -0.5 2 rpy=0 0 0 -> xyz=0 -0.5 1 rpy=0 0 0
- joint Torso_FrontLeg: origin xyz=0 0.5 2 rpy=0 0 0 -> xyz=0 0.5 1 rpy=0 0 0
- joint Torso_LeftLegFirst: origin xyz=-0.5 -0.1 2 rpy=0 0 0 -> xyz=-0.5 -0.1 1 rpy=0 0 0
- joint Torso_LeftLegSecond: origin xyz=-0.5 0.1 2 rpy=0 0 0 -> xyz=-0.5 0.1 1 rpy=0 0 0
- joint Torso_RightLegFirst: origin xyz=0.5 -0.1 2 rpy=0 0 0 -> xyz=0.5 -0.1 1 rpy=0 0 0
- joint Torso_RightLegSecond: origin xyz=0.5 0.1 2 rpy=0 0 0 -> xyz=0.5 0.1 1 rpy=0 0 0

Commit message: updated numpy part b

File: body.urdf (robot description, URDF)
Before this commit: robot robot, 13 links, 12 joints
Links:
- removed link BackLowerLeg
- removed link FrontLowerLeg
- removed link LeftLegFirst
- removed link LeftLegSecond
- removed link LeftLowerLegFirst
- removed link LeftLowerLegSecond
- removed link RightLegFirst
- removed link RightLegSecond
- removed link RightLowerLegFirst
- removed link RightLowerLegSecond
- added link BackLowerleg, mass 1; collision box size=0.2 0.2 1; visual box size=0.2 0.2 1
- added link FrontLowerleg, mass 1; collision box size=0.2 0.2 1; visual box size=0.2 0.2 1
- added link LeftLowerleg, mass 1; collision box size=0.2 0.2 1; visual box size=0.2 0.2 1
- added link Leftleg, mass 1; collision box size=1 0.2 0.2; visual box size=1 0.2 0.2
- added link RightLowerleg, mass 1; collision box size=0.2 0.2 1; visual box size=0.2 0.2 1
- added link Rightleg, mass 1; collision box size=1 0.2 0.2; visual box size=1 0.2 0.2
Joints:
- removed joint BackLeg_BackLowerLeg
- removed joint FrontLeg_FrontLowerLeg
- removed joint LeftLegFirst_LeftLowerLegFirst
- removed joint LeftLegSecond_LeftLowerLegSecond
- removed joint RightLegFirst_RightLowerLegFirst
- removed joint RightLegSecond_RightLowerLegSecond
- removed joint Torso_LeftLegFirst
- removed joint Torso_LeftLegSecond
- removed joint Torso_RightLegFirst
- removed joint Torso_RightLegSecond
- added joint Backleg_BacklowerLeg: type revolute, parent BackLeg, child BackLowerleg, origin xyz=0 -1 0 rpy=0 0 0, axis 1 0 0, limit lower=-3.14159 upper=3.14159 effort=0.0 velocity=0.0
- added joint Frontleg_FrontlowerLeg: type revolute, parent FrontLeg, child FrontLowerleg, origin xyz=0 1 0 rpy=0 0 0, axis 1 0 0, limit lower=-3.14159 upper=3.14159 effort=0.0 velocity=0.0
- added joint Leftleg_Leftlowerleg: type revolute, parent FrontLeg, child LeftLowerleg, origin xyz=-1.5 -0.5 0 rpy=0 0 0, axis 0 1 0, limit lower=-3.14159 upper=3.14159 effort=0.0 velocity=0.0
- added joint Rightleg_RightLowerleg: type revolute, parent Rightleg, child RightLowerleg, origin xyz=1 0 0 rpy=0 0 0, axis 0 1 0, limit lower=-3.14159 upper=3.14159 effort=0.0 velocity=0.0
- added joint Torso_LeftLeg: type revolute, parent Torso, child Leftleg, origin xyz=-0.5 0 1 rpy=0 0 0, axis 0 1 0, limit lower=-3.14159 upper=3.14159 effort=0.0 velocity=0.0
- added joint Torso_RightLeg: type revolute, parent Torso, child Rightleg, origin xyz=0.5 0 1 rpy=0 0 0, axis 0 1 0, limit lower=-3.14159 upper=3.14159 effort=0.0 velocity=0.0

Commit message: quad ped base

File: body.urdf (robot description, URDF)
Before this commit: robot robot, 9 links, 8 joints
Links:
- removed link BackLowerleg
- removed link FrontLowerleg
- removed link LeftLowerleg
- removed link Leftleg
- removed link RightLowerleg
- removed link Rightleg
- link BackLeg: geometry collision box size=1 1 1; visual box size=1 1 1
- link FrontLeg: geometry collision box size=1 1 1; visual box size=1 1 1
Joints:
- removed joint Backleg_BacklowerLeg
- removed joint Frontleg_FrontlowerLeg
- removed joint Leftleg_Leftlowerleg
- removed joint Rightleg_RightLowerleg
- removed joint Torso_LeftLeg
- removed joint Torso_RightLeg
- joint Torso_BackLeg: axis 1 0 0 -> 0 1 0; origin xyz=0 -0.5 1 rpy=0 0 0 -> xyz=1 0 1 rpy=0 0 0
- joint Torso_FrontLeg: axis 1 0 0 -> 0 1 0; origin xyz=0 0.5 1 rpy=0 0 0 -> xyz=2 0 1 rpy=0 0 0
